File: TSA Tracker 04-03-21/TSA Tracker/TSA Location Tracker/TSA Location Tracker.sch (KiCad schematic (older format))
At the start: 15 parts, among them U1 AdafruitCharger

Commit message: Updated switch to push button symbol
Parts:
- Arduino1: symbol Arduino-nano-33:Arduino-NANO-33 -> TSA-Location-Tracker-rescue:Arduino-NANO-33-Arduino-nano-33
- LED_Switch1: symbol Switch:SW_SPST -> Switch:SW_Push
- U1: symbol AdafruitCharger:AdafruitCharger -> TSA-Location-Tracker-rescue:AdafruitCharger-AdafruitCharger
Connections:
- no-connect marks 0 -> 25
Other:
- moved on the sheet: Arduino1, D1, Mode_Switch1, Power_Switch1A, R1, R2, R3, R4, R5, U1
